File: PCB/v1/ReaXtrobe.brd (EAGLE design)
At the start: 59.9 x 15.9 mm, 26 parts, among them J1 OSTVN02A150, J2 OSTVN03A150, U1 ATMEGA328P-AU, U2 NCP1117ST50T3G, U3 MAX9814, Y1 FA-238 16.0000MB-C3

Commit message: V1 BOM
Parts:
- C3: value 100n -> 0.1u
Connections:
- new net N$14: U1.2
- new net N$15: U1.9
- new net N$16: U1.10
- new net N$17: U1.11
- new net N$18: U1.12
- new net N$19: U1.13
Other:
- board text added: "tindie.com/ stores/ neon-cyborg- superstore/"
Changed lines of the file:
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@@
 <drawing>
 <settings>
-<setting alwaysvectorfont="yes"/>
+<setting alwaysvectorfont="no"/>
 <setting verticaltext="up"/>
 </settings>
@@
 </layers>
 <board>
-<fusionsync huburn="a.cGVyc29uYWw6dWUyZGY0M2Ex" projecturn="a.cGVyc29uYWw6dWUyZGY0M2ExIzIwMTkwODExMjA4MTA5ODU2" f3durn="urn:adsk.wipprod:dm.lineage:kkq9xZE2RjqpAUft0sQsQQ" pcbguid="4d4ffd75-ef08-4544-8e3f-84918b628855" lastpulledtime="" lastsyncedchangeguid="39ae548f-6b7b-0a2a-0a14-cb1f4347e5c0"/>
+<fusionsync huburn="a.cGVyc29uYWw6dWUyZGY0M2Ex" projecturn="a.cGVyc29uYWw6dWUyZGY0M2ExIzIwMTkwODExMjA4MTA5ODU2" f3durn="urn:adsk.wipprod:dm.lineage:kkq9xZE2RjqpAUft0sQsQQ" pcbguid="4d4ffd75-ef08-4544-8e3f-84918b628855" lastpulledtime="" lastsyncedchangeguid="1d47761e-0a6c-94a8-aaa3-13c23d44ed40"/>
 <plain>
 <wire x1="0" y1="0" x2="59.924" y2="0" width="0" layer="20"/>
@@
 <vertex x="39.990875" y="9.315028125"/>
 </polygon>
+<text x="52.451" y="8.001" size="1.27" layer="26" font="vector" rot="MR90" align="center">tindie.com/
+stores/
+neon-cyborg-
+superstore/</text>
 </plain>
 <attributes>
@@
 <attribute name="NAME" x="20.701" y="3.556" size="1.27" layer="25" rot="R180"/>
 </element>
-<element name="C3" library="roomready" library_urn="urn:adsk.eagle:library:9911636" package="C0603" package3d_urn="urn:adsk.eagle:package:7587834/2" value="100n" x="31.115" y="13.081" smashed="yes" rot="R180">
+<element name="C3" library="roomready" library_urn="urn:adsk.eagle:library:9911636" package="C0603" package3d_urn="urn:adsk.eagle:package:7587834/2" value="0.1u" x="31.115" y="13.081" smashed="yes" rot="R180">
 <attribute name="NAME" x="34.925" y="13.589" size="1.27" layer="25" rot="R180"/>
 </element>
@@
 <wire x1="37.866" y1="8.236" x2="37.084" y2="7.454" width="0.2032" layer="1"/>
 </signal>
+<signal name="N$14">
+<contactref element="U1" pad="2"/>
+</signal>
+<signal name="N$15">
+<contactref element="U1" pad="9"/>
+</signal>
+<signal name="N$16">
+<contactref element="U1" pad="10"/>
+</signal>
+<signal name="N$17">
+<contactref element="U1" pad="11"/>
+</signal>
+<signal name="N$18">
+<contactref element="U1" pad="12"/>
+</signal>
+<signal name="N$19">
+<contactref element="U1" pad="13"/>
+</signal>
 </signals>
 <mfgpreviewcolors>
@@
 </drawing>
 <compatibility>
+<note version="6.3" minversion="6.2.2" severity="warning">
+Since Version 6.2.2 text objects can contain more than one line,
+which will not be processed correctly with this version.
+</note>
 <note version="8.2" severity="warning">
 Since Version 8.2, EAGLE supports online libraries. The ids
