File: PCB/v1/ReaXtrobe.sch (EAGLE design)
At the start: 26 parts, among them J1 OSTVN02A150, J2 OSTVN03A150, U1 ATMEGA328P-AU, U2 NCP1117ST50T3G, U3 MAX9814, Y1 FA-238 16.0000MB-C3

Commit message: V1 BOM
Parts:
- C3: value 100n -> 0.1u
Connections:
- new net N$14: U1.PD4(XCK/T0)
- new net N$15: U1.PD5(T1)
- new net N$16: U1.PD6(AIN0)
- new net N$17: U1.PD7(AIN1)
- new net N$18: U1.PB0(ICP)
- new net N$19: U1.PB1(OC1A)
Changed lines of the file:
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@@
 <part name="GND2" library="supply1" library_urn="urn:adsk.eagle:library:371" deviceset="GND" device=""/>
 <part name="R1" library="roomready" library_urn="urn:adsk.eagle:library:9911636" deviceset="RES-SMD" device="0603" package3d_urn="urn:adsk.eagle:package:7587835/3" value="1k"/>
-<part name="C3" library="roomready" library_urn="urn:adsk.eagle:library:9911636" deviceset="CAP-CER-SMD" device="0603" package3d_urn="urn:adsk.eagle:package:7587834/2" value="100n"/>
+<part name="C3" library="roomready" library_urn="urn:adsk.eagle:library:9911636" deviceset="CAP-CER-SMD" device="0603" package3d_urn="urn:adsk.eagle:package:7587834/2" value="0.1u"/>
 <part name="GND3" library="supply1" library_urn="urn:adsk.eagle:library:371" deviceset="GND" device=""/>
 <part name="C4" library="roomready" library_urn="urn:adsk.eagle:library:9911636" deviceset="CAP-CER-SMD" device="0603" package3d_urn="urn:adsk.eagle:package:7587834/2" value="1u"/>
@@
 </segment>
 </net>
+<net name="N$14" class="0">
+<segment>
+<pinref part="U1" gate="G$1" pin="PD4(XCK/T0)"/>
+<wire x1="182.88" y1="119.38" x2="193.04" y2="119.38" width="0.1524" layer="91"/>
+</segment>
+</net>
+<net name="N$15" class="0">
+<segment>
+<pinref part="U1" gate="G$1" pin="PD5(T1)"/>
+<wire x1="182.88" y1="121.92" x2="193.04" y2="121.92" width="0.1524" layer="91"/>
+</segment>
+</net>
+<net name="N$16" class="0">
+<segment>
+<pinref part="U1" gate="G$1" pin="PD6(AIN0)"/>
+<wire x1="182.88" y1="124.46" x2="193.04" y2="124.46" width="0.1524" layer="91"/>
+</segment>
+</net>
+<net name="N$17" class="0">
+<segment>
+<pinref part="U1" gate="G$1" pin="PD7(AIN1)"/>
+<wire x1="182.88" y1="127" x2="193.04" y2="127" width="0.1524" layer="91"/>
+</segment>
+</net>
+<net name="N$18" class="0">
+<segment>
+<pinref part="U1" gate="G$1" pin="PB0(ICP)"/>
+<wire x1="182.88" y1="149.86" x2="193.04" y2="149.86" width="0.1524" layer="91"/>
+</segment>
+</net>
+<net name="N$19" class="0">
+<segment>
+<pinref part="U1" gate="G$1" pin="PB1(OC1A)"/>
+<wire x1="182.88" y1="152.4" x2="193.04" y2="152.4" width="0.1524" layer="91"/>
+</segment>
+</net>
